Commit message: tried to make urdf file work

File: hexapod/hexapod/urdf/hexapod_description.xacro (robot description, xacro)
@@ -1,5 +1,5 @@
 <?xml version="1.0" ?>
 <robot name="hexapod" xmlns:xacro="http://www.ros.org/wiki/xacro">
-<xacro:include filename="/home/darsh/Desktop/ROS/Hexapod/hexapod/urdf/materials.xacro" />
+<xacro:include filename="materials.xacro" />
 <link name="base_link">
   <inertial>
@@ -11,5 +11,5 @@
     <origin xyz="0 0 0" rpy="0 0 0"/>
     <geometry>
-      <mesh filename="/home/darsh/Desktop/ROS/Hexapod/hexapod/meshes/base_link.stl" scale="0.001 0.001 0.001"/>
+      <mesh filename="package://hexapod/meshes/base_link.stl" scale="0.001 0.001 0.001"/>
     </geometry>
     <material name="silver"/>
@@ -18,5 +18,5 @@
     <origin xyz="0 0 0" rpy="0 0 0"/>
     <geometry>
-      <mesh filename="/home/darsh/Desktop/ROS/Hexapod/hexapod/meshes/base_link.stl" scale="0.001 0.001 0.001"/>
+      <mesh filename="package://hexapod/meshes/base_link.stl" scale="0.001 0.001 0.001"/>
     </geometry>
   </collision>
@@ -31,5 +31,5 @@
     <origin xyz="0.043597 0.082619 0.0021" rpy="0 0 0"/>
     <geometry>
-      <mesh filename="/home/darsh/Desktop/ROS/Hexapod/hexapod/meshes/link_1_v1_1_6.stl" scale="0.001 0.001 0.001"/>
+      <mesh filename="package://hexapod/meshes/link_1_v1_1_6.stl" scale="0.001 0.001 0.001"/>
     </geometry>
     <material name="silver"/>
@@ -38,5 +38,5 @@
     <origin xyz="0.043597 0.082619 0.0021" rpy="0 0 0"/>
     <geometry>
-      <mesh filename="/home/darsh/Desktop/ROS/Hexapod/hexapod/meshes/link_1_v1_1_6.stl" scale="0.001 0.001 0.001"/>
+      <mesh filename="package://hexapod/meshes/link_1_v1_1_6.stl" scale="0.001 0.001 0.001"/>
     </geometry>
   </collision>
@@ -51,5 +51,5 @@
     <origin xyz="-0.044403 0.082619 0.0021" rpy="0 0 0"/>
     <geometry>
-      <mesh filename="/home/darsh/Desktop/ROS/Hexapod/hexapod/meshes/link_1_v1_1_1.stl" scale="0.001 0.001 0.001"/>
+      <mesh filename="package://hexapod/meshes/link_1_v1_1_1.stl" scale="0.001 0.001 0.001"/>
     </geometry>
     <material name="silver"/>
@@ -58,5 +58,5 @@
     <origin xyz="-0.044403 0.082619 0.0021" rpy="0 0 0"/>
     <geometry>
-      <mesh filename="/home/darsh/Desktop/ROS/Hexapod/hexapod/meshes/link_1_v1_1_1.stl" scale="0.001 0.001 0.001"/>
+      <mesh filename="package://hexapod/meshes/link_1_v1_1_1.stl" scale="0.001 0.001 0.001"/>
     </geometry>
   </collision>
@@ -71,5 +71,5 @@
     <origin xyz="-0.088403 0.006409 0.0021" rpy="0 0 0"/>
     <geometry>
-      <mesh filename="/home/darsh/Desktop/ROS/Hexapod/hexapod/meshes/link_1_v1_1_4.stl" scale="0.001 0.001 0.001"/>
+      <mesh filename="package://hexapod/meshes/link_1_v1_1_4.stl" scale="0.001 0.001 0.001"/>
     </geometry>
     <material name="silver"/>
@@ -78,5 +78,5 @@
     <origin xyz="-0.088403 0.006409 0.0021" rpy="0 0 0"/>
     <geometry>
-      <mesh filename="/home/darsh/Desktop/ROS/Hexapod/hexapod/meshes/link_1_v1_1_4.stl" scale="0.001 0.001 0.001"/>
+      <mesh filename="package://hexapod/meshes/link_1_v1_1_4.stl" scale="0.001 0.001 0.001"/>
     </geometry>
   </collision>
@@ -91,5 +91,5 @@
     <origin xyz="-0.044403 -0.069802 0.0021" rpy="0 0 0"/>
     <geometry>
-      <mesh filename="/home/darsh/Desktop/ROS/Hexapod/hexapod/meshes/link_1_v1_1_2.stl" scale="0.001 0.001 0.001"/>
+      <mesh filename="package://hexapod/meshes/link_1_v1_1_2.stl" scale="0.001 0.001 0.001"/>
     </geometry>
     <material name="silver"/>
@@ -98,5 +98,5 @@
     <origin xyz="-0.044403 -0.069802 0.0021" rpy="0 0 0"/>
     <geometry>
-      <mesh filename="/home/darsh/Desktop/ROS/Hexapod/hexapod/meshes/link_1_v1_1_2.stl" scale="0.001 0.001 0.001"/>
+      <mesh filename="package://hexapod/meshes/link_1_v1_1_2.stl" scale="0.001 0.001 0.001"/>
     </geometry>
   </collision>
@@ -111,5 +111,5 @@
     <origin xyz="0.043597 -0.069802 0.0021" rpy="0 0 0"/>
     <geometry>
-      <mesh filename="/home/darsh/Desktop/ROS/Hexapod/hexapod/meshes/link_1_v1_1_3.stl" scale="0.001 0.001 0.001"/>
+      <mesh filename="package://hexapod/meshes/link_1_v1_1_3.stl" scale="0.001 0.001 0.001"/>
     </geometry>
     <material name="silver"/>
@@ -118,5 +118,5 @@
     <origin xyz="0.043597 -0.069802 0.0021" rpy="0 0 0"/>
     <geometry>
-      <mesh filename="/home/darsh/Desktop/ROS/Hexapod/hexapod/meshes/link_1_v1_1_3.stl" scale="0.001 0.001 0.001"/>
+      <mesh filename="package://hexapod/meshes/link_1_v1_1_3.stl" scale="0.001 0.001 0.001"/>
     </geometry>
   </collision>
@@ -131,5 +131,5 @@
     <origin xyz="0.089297 0.006409 0.0021" rpy="0 0 0"/>
     <geometry>
-      <mesh filename="/home/darsh/Desktop/ROS/Hexapod/hexapod/meshes/link_1_v1_1_5.stl" scale="0.001 0.001 0.001"/>
+      <mesh filename="package://hexapod/meshes/link_1_v1_1_5.stl" scale="0.001 0.001 0.001"/>
     </geometry>
     <material name="silver"/>
@@ -138,5 +138,5 @@
     <origin xyz="0.089297 0.006409 0.0021" rpy="0 0 0"/>
     <geometry>
-      <mesh filename="/home/darsh/Desktop/ROS/Hexapod/hexapod/meshes/link_1_v1_1_5.stl" scale="0.001 0.001 0.001"/>
+      <mesh filename="package://hexapod/meshes/link_1_v1_1_5.stl" scale="0.001 0.001 0.001"/>
     </geometry>
   </collision>
@@ -151,5 +151,5 @@
     <origin xyz="-0.095156 0.10997 -0.0244" rpy="0 0 0"/>
     <geometry>
-      <mesh filename="/home/darsh/Desktop/ROS/Hexapod/hexapod/meshes/link_2_v1_1_1.stl" scale="0.001 0.001 0.001"/>
+      <mesh filename="package://hexapod/meshes/link_2_v1_1_1.stl" scale="0.001 0.001 0.001"/>
     </geometry>
     <material name="silver"/>
@@ -158,5 +158,5 @@
     <origin xyz="-0.095156 0.10997 -0.0244" rpy="0 0 0"/>
     <geometry>
-      <mesh filename="/home/darsh/Desktop/ROS/Hexapod/hexapod/meshes/link_2_v1_1_1.stl" scale="0.001 0.001 0.001"/>
+      <mesh filename="package://hexapod/meshes/link_2_v1_1_1.stl" scale="0.001 0.001 0.001"/>
     </geometry>
   </collision>
@@ -171,5 +171,5 @@
     <origin xyz="-0.139245 -0.020778 -0.0244" rpy="0 0 0"/>
     <geometry>
-      <mesh filename="/home/darsh/Desktop/ROS/Hexapod/hexapod/meshes/link_2_v1_1_2.stl" scale="0.001 0.001 0.001"/>
+      <mesh filename="package://hexapod/meshes/link_2_v1_1_2.stl" scale="0.001 0.001 0.001"/>
     </geometry>
     <material name="silver"/>
@@ -178,5 +178,5 @@
     <origin xyz="-0.139245 -0.020778 -0.0244" rpy="0 0 0"/>
     <geometry>
-      <mesh filename="/home/darsh/Desktop/ROS/Hexapod/hexapod/meshes/link_2_v1_1_2.stl" scale="0.001 0.001 0.001"/>
+      <mesh filename="package://hexapod/meshes/link_2_v1_1_2.stl" scale="0.001 0.001 0.001"/>
     </geometry>
   </collision>
@@ -191,5 +191,5 @@
     <origin xyz="0.051014 0.139794 -0.0244" rpy="0 0 0"/>
     <geometry>
-      <mesh filename="/home/darsh/Desktop/ROS/Hexapod/hexapod/meshes/link_2_v1_1_6.stl" scale="0.001 0.001 0.001"/>
+      <mesh filename="package://hexapod/meshes/link_2_v1_1_6.stl" scale="0.001 0.001 0.001"/>
     </geometry>
     <material name="silver"/>
@@ -198,5 +198,5 @@
     <origin xyz="0.051014 0.139794 -0.0244" rpy="0 0 0"/>
     <geometry>
-      <mesh filename="/home/darsh/Desktop/ROS/Hexapod/hexapod/meshes/link_2_v1_1_6.stl" scale="0.001 0.001 0.001"/>
+      <mesh filename="package://hexapod/meshes/link_2_v1_1_6.stl" scale="0.001 0.001 0.001"/>
     </geometry>
   </collision>
@@ -211,5 +211,5 @@
     <origin xyz="-0.048131 -0.127335 -0.0244" rpy="0 0 0"/>
     <geometry>
-      <mesh filename="/home/darsh/Desktop/ROS/Hexapod/hexapod/meshes/link_2_v1_1_4.stl" scale="0.001 0.001 0.001"/>
+      <mesh filename="package://hexapod/meshes/link_2_v1_1_4.stl" scale="0.001 0.001 0.001"/>
     </geometry>
     <material name="silver"/>
@@ -218,5 +218,5 @@
     <origin xyz="-0.048131 -0.127335 -0.0244" rpy="0 0 0"/>
     <geometry>
-      <mesh filename="/home/darsh/Desktop/ROS/Hexapod/hexapod/meshes/link_2_v1_1_4.stl" scale="0.001 0.001 0.001"/>
+      <mesh filename="package://hexapod/meshes/link_2_v1_1_4.stl" scale="0.001 0.001 0.001"/>
     </geometry>
   </collision>
@@ -231,5 +231,5 @@
     <origin xyz="0.093119 -0.099325 -0.0244" rpy="0 0 0"/>
     <geometry>
-      <mesh filename="/home/darsh/Desktop/ROS/Hexapod/hexapod/meshes/link_2_v1_1_5.stl" scale="0.001 0.001 0.001"/>
+      <mesh filename="package://hexapod/meshes/link_2_v1_1_5.stl" scale="0.001 0.001 0.001"/>
     </geometry>
     <material name="silver"/>
@@ -238,5 +238,5 @@
     <origin xyz="0.093119 -0.099325 -0.0244" rpy="0 0 0"/>
     <geometry>
-      <mesh filename="/home/darsh/Desktop/ROS/Hexapod/hexapod/meshes/link_2_v1_1_5.stl" scale="0.001 0.001 0.001"/>
+      <mesh filename="package://hexapod/meshes/link_2_v1_1_5.stl" scale="0.001 0.001 0.001"/>
     </geometry>
   </collision>
@@ -251,5 +251,5 @@
     <origin xyz="0.141258 -0.020168 -0.0244" rpy="0 0 0"/>
     <geometry>
-      <mesh filename="/home/darsh/Desktop/ROS/Hexapod/hexapod/meshes/link_2_v1_1_3.stl" scale="0.001 0.001 0.001"/>
+      <mesh filename="package://hexapod/meshes/link_2_v1_1_3.stl" scale="0.001 0.001 0.001"/>
     </geometry>
     <material name="silver"/>
@@ -258,5 +258,5 @@
     <origin xyz="0.141258 -0.020168 -0.0244" rpy="0 0 0"/>
     <geometry>
-      <mesh filename="/home/darsh/Desktop/ROS/Hexapod/hexapod/meshes/link_2_v1_1_3.stl" scale="0.001 0.001 0.001"/>
+      <mesh filename="package://hexapod/meshes/link_2_v1_1_3.stl" scale="0.001 0.001 0.001"/>
     </geometry>
   </collision>
@@ -271,5 +271,5 @@
     <origin xyz="-0.23747 0.027103 -0.0244" rpy="0 0 0"/>
     <geometry>
-      <mesh filename="/home/darsh/Desktop/ROS/Hexapod/hexapod/meshes/L3_v4_1_2.stl" scale="0.001 0.001 0.001"/>
+      <mesh filename="package://hexapod/meshes/L3_v4_1_2.stl" scale="0.001 0.001 0.001"/>
     </geometry>
     <material name="silver"/>
@@ -278,5 +278,5 @@
     <origin xyz="-0.23747 0.027103 -0.0244" rpy="0 0 0"/>
     <geometry>
-      <mesh filename="/home/darsh/Desktop/ROS/Hexapod/hexapod/meshes/L3_v4_1_2.stl" scale="0.001 0.001 0.001"/>
+      <mesh filename="package://hexapod/meshes/L3_v4_1_2.stl" scale="0.001 0.001 0.001"/>
     </geometry>
   </collision>
@@ -291,5 +291,5 @@
     <origin xyz="-0.095321 -0.210936 -0.0244" rpy="0 0 0"/>
     <geometry>
-      <mesh filename="/home/darsh/Desktop/ROS/Hexapod/hexapod/meshes/L3_v4_1_3.stl" scale="0.001 0.001 0.001"/>
+      <mesh filename="package://hexapod/meshes/L3_v4_1_3.stl" scale="0.001 0.001 0.001"/>
     </geometry>
     <material name="silver"/>
@@ -298,5 +298,5 @@
     <origin xyz="-0.095321 -0.210936 -0.0244" rpy="0 0 0"/>
     <geometry>
-      <mesh filename="/home/darsh/Desktop/ROS/Hexapod/hexapod/meshes/L3_v4_1_3.stl" scale="0.001 0.001 0.001"/>
+      <mesh filename="package://hexapod/meshes/L3_v4_1_3.stl" scale="0.001 0.001 0.001"/>
     </geometry>
   </collision>
@@ -311,5 +311,5 @@
     <origin xyz="0.146259 -0.179276 -0.0244" rpy="0 0 0"/>
     <geometry>
-      <mesh filename="/home/darsh/Desktop/ROS/Hexapod/hexapod/meshes/L3_v4_1_6.stl" scale="0.001 0.001 0.001"/>
+      <mesh filename="package://hexapod/meshes/L3_v4_1_6.stl" scale="0.001 0.001 0.001"/>
     </geometry>
     <material name="silver"/>
@@ -318,5 +318,5 @@
     <origin xyz="0.146259 -0.179276 -0.0244" rpy="0 0 0"/>
     <geometry>
-      <mesh filename="/home/darsh/Desktop/ROS/Hexapod/hexapod/meshes/L3_v4_1_6.stl" scale="0.001 0.001 0.001"/>
+      <mesh filename="package://hexapod/meshes/L3_v4_1_6.stl" scale="0.001 0.001 0.001"/>
     </geometry>
   </collision>
@@ -331,5 +331,5 @@
     <origin xyz="0.237335 0.031891 -0.0244" rpy="0 0 0"/>
     <geometry>
-      <mesh filename="/home/darsh/Desktop/ROS/Hexapod/hexapod/meshes/L3_v4_1_5.stl" scale="0.001 0.001 0.001"/>
+      <mesh filename="package://hexapod/meshes/L3_v4_1_5.stl" scale="0.001 0.001 0.001"/>
     </geometry>
     <material name="silver"/>
@@ -338,5 +338,5 @@
     <origin xyz="0.237335 0.031891 -0.0244" rpy="0 0 0"/>
     <geometry>
-      <mesh filename="/home/darsh/Desktop/ROS/Hexapod/hexapod/meshes/L3_v4_1_5.stl" scale="0.001 0.001 0.001"/>
+      <mesh filename="package://hexapod/meshes/L3_v4_1_5.stl" scale="0.001 0.001 0.001"/>
     </geometry>
   </collision>
@@ -351,5 +351,5 @@
     <origin xyz="0.147058 0.191913 -0.0244" rpy="0 0 0"/>
     <geometry>
-      <mesh filename="/home/darsh/Desktop/ROS/Hexapod/hexapod/meshes/L3_v4_1_4.stl" scale="0.001 0.001 0.001"/>
+      <mesh filename="package://hexapod/meshes/L3_v4_1_4.stl" scale="0.001 0.001 0.001"/>
     </geometry>
     <material name="silver"/>
@@ -358,5 +358,5 @@
     <origin xyz="0.147058 0.191913 -0.0244" rpy="0 0 0"/>
     <geometry>
-      <mesh filename="/home/darsh/Desktop/ROS/Hexapod/hexapod/meshes/L3_v4_1_4.stl" scale="0.001 0.001 0.001"/>
+      <mesh filename="package://hexapod/meshes/L3_v4_1_4.stl" scale="0.001 0.001 0.001"/>
     </geometry>
   </collision>
@@ -371,5 +371,5 @@
     <origin xyz="-0.063545 -0.030046 -0.026" rpy="0 0 0"/>
     <geometry>
-      <mesh filename="/home/darsh/Desktop/ROS/Hexapod/hexapod/meshes/Top_plate_v2_1.stl" scale="0.001 0.001 0.001"/>
+      <mesh filename="package://hexapod/meshes/Top_plate_v2_1.stl" scale="0.001 0.001 0.001"/>
     </geometry>
     <material name="silver"/>
@@ -378,5 +378,5 @@
     <origin xyz="-0.063545 -0.030046 -0.026" rpy="0 0 0"/>
     <geometry>
-      <mesh filename="/home/darsh/Desktop/ROS/Hexapod/hexapod/meshes/Top_plate_v2_1.stl" scale="0.001 0.001 0.001"/>
+      <mesh filename="package://hexapod/meshes/Top_plate_v2_1.stl" scale="0.001 0.001 0.001"/>
     </geometry>
   </collision>

File: hexapod/hexapod/urdf/robot_description.urdf (robot description, URDF)
Before this commit: robot hexapod, 19 links, 18 joints
Links:
- link L3_v4_1_2: geometry collision mesh filename=file://$(find hexapod)/meshes/L3_v4_1_2.stl scale=0.001 0.001 0.001; visual mesh filename=file://$(find hexapod)/meshes/L3_v4_1_2.stl scale=0.001 0.001 0.001
- link L3_v4_1_3: geometry collision mesh filename=file://$(find hexapod)/meshes/L3_v4_1_3.stl scale=0.001 0.001 0.001; visual mesh filename=file://$(find hexapod)/meshes/L3_v4_1_3.stl scale=0.001 0.001 0.001
- link L3_v4_1_4: geometry collision mesh filename=file://$(find hexapod)/meshes/L3_v4_1_4.stl scale=0.001 0.001 0.001; visual mesh filename=file://$(find hexapod)/meshes/L3_v4_1_4.stl scale=0.001 0.001 0.001
- link L3_v4_1_5: geometry collision mesh filename=file://$(find hexapod)/meshes/L3_v4_1_5.stl scale=0.001 0.001 0.001; visual mesh filename=file://$(find hexapod)/meshes/L3_v4_1_5.stl scale=0.001 0.001 0.001
- link L3_v4_1_6: geometry collision mesh filename=file://$(find hexapod)/meshes/L3_v4_1_6.stl scale=0.001 0.001 0.001; visual mesh filename=file://$(find hexapod)/meshes/L3_v4_1_6.stl scale=0.001 0.001 0.001
- link Top_plate_v2_1: geometry collision mesh filename=file://$(find hexapod)/meshes/Top_plate_v2_1.stl scale=0.001 0.001 0.001; visual mesh filename=file://$(find hexapod)/meshes/Top_plate_v2_1.stl scale=0.001 0.001 0.001
- link base_link: geometry collision mesh filename=file://$(find hexapod)/meshes/base_link.stl scale=0.001 0.001 0.001; visual mesh filename=file://$(find hexapod)/meshes/base_link.stl scale=0.001 0.001 0.001
- link link_1_v1_1_1: geometry collision mesh filename=file://$(find hexapod)/meshes/link_1_v1_1_1.stl scale=0.001 0.001 0.001; visual mesh filename=file://$(find hexapod)/meshes/link_1_v1_1_1.stl scale=0.001 0.001 0.001
- link link_1_v1_1_2: geometry collision mesh filename=file://$(find hexapod)/meshes/link_1_v1_1_2.stl scale=0.001 0.001 0.001; visual mesh filename=file://$(find hexapod)/meshes/link_1_v1_1_2.stl scale=0.001 0.001 0.001
- link link_1_v1_1_3: geometry collision mesh filename=file://$(find hexapod)/meshes/link_1_v1_1_3.stl scale=0.001 0.001 0.001; visual mesh filename=file://$(find hexapod)/meshes/link_1_v1_1_3.stl scale=0.001 0.001 0.001
- link link_1_v1_1_4: geometry collision mesh filename=file://$(find hexapod)/meshes/link_1_v1_1_4.stl scale=0.001 0.001 0.001; visual mesh filename=file://$(find hexapod)/meshes/link_1_v1_1_4.stl scale=0.001 0.001 0.001
- link link_1_v1_1_5: geometry collision mesh filename=file://$(find hexapod)/meshes/link_1_v1_1_5.stl scale=0.001 0.001 0.001; visual mesh filename=file://$(find hexapod)/meshes/link_1_v1_1_5.stl scale=0.001 0.001 0.001
- link link_1_v1_1_6: geometry collision mesh filename=file://$(find hexapod)/meshes/link_1_v1_1_6.stl scale=0.001 0.001 0.001; visual mesh filename=file://$(find hexapod)/meshes/link_1_v1_1_6.stl scale=0.001 0.001 0.001
- link link_2_v1_1_1: geometry collision mesh filename=file://$(find hexapod)/meshes/link_2_v1_1_1.stl scale=0.001 0.001 0.001; visual mesh filename=file://$(find hexapod)/meshes/link_2_v1_1_1.stl scale=0.001 0.001 0.001
- link link_2_v1_1_2: geometry collision mesh filename=file://$(find hexapod)/meshes/link_2_v1_1_2.stl scale=0.001 0.001 0.001; visual mesh filename=file://$(find hexapod)/meshes/link_2_v1_1_2.stl scale=0.001 0.001 0.001
- link link_2_v1_1_3: geometry collision mesh filename=file://$(find hexapod)/meshes/link_2_v1_1_3.stl scale=0.001 0.001 0.001; visual mesh filename=file://$(find hexapod)/meshes/link_2_v1_1_3.stl scale=0.001 0.001 0.001
- link link_2_v1_1_4: geometry collision mesh filename=file://$(find hexapod)/meshes/link_2_v1_1_4.stl scale=0.001 0.001 0.001; visual mesh filename=file://$(find hexapod)/meshes/link_2_v1_1_4.stl scale=0.001 0.001 0.001
- link link_2_v1_1_5: geometry collision mesh filename=file://$(find hexapod)/meshes/link_2_v1_1_5.stl scale=0.001 0.001 0.001; visual mesh filename=file://$(find hexapod)/meshes/link_2_v1_1_5.stl scale=0.001 0.001 0.001
- link link_2_v1_1_6: geometry collision mesh filename=file://$(find hexapod)/meshes/link_2_v1_1_6.stl scale=0.001 0.001 0.001; visual mesh filename=file://$(find hexapod)/meshes/link_2_v1_1_6.stl scale=0.001 0.001 0.001
